File: Production_Files/circuit-boards/kicad/calliope-mirror-heater/calliope-mirror-heater.kicad_pcb (KiCad board)
At the start: 2 copper layers, 1 part, among them J101 Conn_02x15_Odd_Even

Commit message: Electrically done
Parts:
- added C101: 100n/16V, Capacitor_SMD:C_0402_1005Metric, F.Cu at (126.1, 92.8)
- added C102: 100n/16V, Capacitor_SMD:C_0402_1005Metric, F.Cu at (106.9, 97.2)
- added C103: 22u/25V, Capacitor_SMD:C_0805_2012Metric, F.Cu at (114.2, 82.1)
- added C401: 22u/25V, Capacitor_SMD:C_0805_2012Metric, F.Cu at (116.5, 86.7)
- added C405: 1u/25V, Capacitor_SMD:C_0402_1005Metric, F.Cu at (112.6, 87.0)
- added D101: H5VL10B, Diode_SMD:D_SOD-882D, F.Cu at (126.0, 89.3)
- added D102: SS34, Diode_SMD:D_SMA, F.Cu at (117.8, 90.5)
- added D103: yellow_heater-energized, LED_SMD:LED_0805_2012Metric, F.Cu at (88.0, 86.6)
- added D104: yellow_heater-energized, LED_SMD:LED_0805_2012Metric, F.Cu at (88.0, 88.5)
- added D105: SS34, Diode_SMD:D_SMA, F.Cu at (123.2, 89.2)
- added D106: H3V3L10B, Diode_SMD:D_SOD-882D, F.Cu at (100.8, 81.8)
- added D107: SS34, Diode_SMD:D_SMA, F.Cu at (102.9, 86.0)
- added D108: SS34, Diode_SMD:D_SMA, F.Cu at (108.2, 85.7)
- added D109: H5VL10B, Diode_SMD:D_SOD-882D, F.Cu at (92.8, 86.3)
- added D1904: H3V3L10B, Diode_SMD:D_SOD-882D, F.Cu at (104.2, 81.8)
- added D1905: H5VL10B, Diode_SMD:D_SOD-882D, F.Cu at (91.0, 88.7)
- added J102: USB_C_Receptacle_USB2.0_16P, Connector_USB:USB_C_Receptacle_GCT_USB4105-xx-A_16P_TopMnt_Horizontal, F.Cu at (131.3, 86.5)
- added R101: Heater-trace_16R_length-6m_width-0.2mm, TestPoint:TestPoint_2Pads_Pitch5.08mm_Drill1.3mm, F.Cu at (116.1, 94.1)
- added R102: 49.9k, Resistor_SMD:R_0402_1005Metric, F.Cu at (119.7, 97.3)
- added R103: 5.1k, Resistor_SMD:R_0402_1005Metric, F.Cu at (126.1, 87.5)
- added R105: 27k, Resistor_SMD:R_0402_1005Metric, F.Cu at (105.7, 94.2)
- added R106: 2.4k, Resistor_SMD:R_0402_1005Metric, F.Cu at (104.7, 94.2)
- added R107: 150, Resistor_SMD:R_0402_1005Metric, F.Cu at (107.8, 97.2)
- added R108: 5.1k, Resistor_SMD:R_0402_1005Metric, F.Cu at (126.1, 85.6)
- added R109: 2.2k, Resistor_SMD:R_0402_1005Metric, F.Cu at (90.2, 86.5)
- added R110: 2.4k, Resistor_SMD:R_0402_1005Metric, F.Cu at (105.7, 88.9)
- added R111: 330, Resistor_SMD:R_0402_1005Metric, F.Cu at (105.7, 87.9)
- added SW102: select-heater-power-source, dpdt-slide-switch:SW_DPDT_shou-han_MST-22D18G2-BD-125, F.Cu at (120.7, 83.4)
- added TH101: 100k_NCP15WF104F03RC, Resistor_SMD:R_0402_1005Metric, F.Cu at (117.6, 99.3)
- added TP101: USB_CC1, testpoint_solid-zone-connection_lib:TestPoint_Pad_D1.0mm, B.Cu at (126.6, 87.2)
- added TP102: USB_CC2, testpoint_solid-zone-connection_lib:TestPoint_Pad_D1.0mm, B.Cu at (127.3, 85.2)
- added TP103: USB_DN, testpoint_solid-zone-connection_lib:TestPoint_Pad_D1.0mm, B.Cu at (129.8, 87.5)
- added TP104: USB_DP, testpoint_solid-zone-connection_lib:TestPoint_Pad_D1.0mm, B.Cu at (129.8, 85.5)
- added TP105: TestPoint_Small, testpoint_solid-zone-connection_lib:TestPoint_Pad_D1.0mm, B.Cu at (121.8, 90.2)
- added TP106: TestPoint_Small, testpoint_solid-zone-connection_lib:TestPoint_Pad_D1.0mm, B.Cu at (126.6, 89.3)
- added TP107: TestPoint_Small, testpoint_solid-zone-connection_lib:TestPoint_Pad_D1.0mm, B.Cu at (106.1, 93.8)
- added TP108: TestPoint_Small, testpoint_solid-zone-connection_lib:TestPoint_Pad_D1.0mm, B.Cu at (107.0, 97.5)
- added TP109: TestPoint_Small, testpoint_solid-zone-connection_lib:TestPoint_Pad_D1.0mm, B.Cu at (106.1, 86.8)
- added TP110: TestPoint_Small, testpoint_solid-zone-connection_lib:TestPoint_Pad_D1.0mm, B.Cu at (105.2, 89.8)
- added TP111: TestPoint_Small, testpoint_solid-zone-connection_lib:TestPoint_Pad_D1.0mm, B.Cu at (107.2, 91.1)
- added TP112: TestPoint_Small, testpoint_solid-zone-connection_lib:TestPoint_Pad_D1.0mm, B.Cu at (114.0, 88.3)
- added TP113: TestPoint_Small, testpoint_solid-zone-connection_lib:TestPoint_Pad_D1.0mm, B.Cu at (112.1, 90.9)
- added TP114: TestPoint_Small, testpoint_solid-zone-connection_lib:TestPoint_Pad_D1.0mm, B.Cu at (120.8, 96.1)
- added TP115: TestPoint_Small, testpoint_solid-zone-connection_lib:TestPoint_Pad_D1.0mm, B.Cu at (122.3, 94.7)
- added TP116: TestPoint_Small, testpoint_solid-zone-connection_lib:TestPoint_Pad_D1.0mm, B.Cu at (121.0, 98.1)
- added TP117: TestPoint_Small, testpoint_solid-zone-connection_lib:TestPoint_Pad_D1.0mm, B.Cu at (126.8, 95.3)
- added TP118: TestPoint_Small, testpoint_solid-zone-connection_lib:TestPoint_Pad_D1.0mm, B.Cu at (126.1, 98.1)
- added TP119: TestPoint_Small, testpoint_solid-zone-connection_lib:TestPoint_Pad_D1.0mm, B.Cu at (127.8, 97.0)
- added TP120: TestPoint_Small, testpoint_solid-zone-connection_lib:TestPoint_Pad_D1.0mm, B.Cu at (115.0, 96.9)
- added TP121: TestPoint_Small, testpoint_solid-zone-connection_lib:TestPoint_Pad_D1.0mm, B.Cu at (91.0, 86.3)
- added TP122: TestPoint_Small, testpoint_solid-zone-connection_lib:TestPoint_Pad_D1.0mm, B.Cu at (118.9, 83.4)
- added TP123: TestPoint_Small, testpoint_solid-zone-connection_lib:TestPoint_Pad_D1.0mm, B.Cu at (118.9, 81.3)
- added TP124: TestPoint_Small, testpoint_solid-zone-connection_lib:TestPoint_Pad_D1.0mm, B.Cu at (120.7, 84.4)
- added TP125: TestPoint_Small, testpoint_solid-zone-connection_lib:TestPoint_Pad_D1.0mm, B.Cu at (120.7, 82.3)
- added TP126: TestPoint_Small, testpoint_solid-zone-connection_lib:TestPoint_Pad_D1.0mm, B.Cu at (123.4, 85.7)
- added TP127: TestPoint_Small, testpoint_solid-zone-connection_lib:TestPoint_Pad_D1.0mm, B.Cu at (123.2, 82.4)
- added TP128: TestPoint_Small, testpoint_solid-zone-connection_lib:TestPoint_Pad_D1.0mm, B.Cu at (126.1, 92.6)
- added TP129: TestPoint_Small, testpoint_solid-zone-connection_lib:TestPoint_Pad_D1.0mm, B.Cu at (124.4, 97.1)
- added TP401: TestPoint_Small, testpoint_solid-zone-connection_lib:TestPoint_Pad_D1.0mm, B.Cu at (116.7, 87.9)
- added TP402: TestPoint_Small, testpoint_solid-zone-connection_lib:TestPoint_Pad_D1.0mm, B.Cu at (113.8, 84.8)
- added TP403: TestPoint_Small, testpoint_solid-zone-connection_lib:TestPoint_Pad_D1.0mm, B.Cu at (111.5, 84.5)
- added U102: LM358DR2G, Package_SO:SOIC-8_3.9x4.9mm_P1.27mm, F.Cu at (123.9, 95.9)
- added U104: TP5709S5, Package_TO_SOT_SMD:SOT-23-5, F.Cu at (104.7, 97.2)
- added U105: GAQY212GSX, Package_SO:SO-4_4.4x4.3mm_P2.54mm, F.Cu at (110.5, 89.8)
- added U401: XC6206P332MR-G, Package_TO_SOT_SMD:SOT-23-3, F.Cu at (113.8, 84.8)
- moved J101 44.6 mm to (97.2, 79.3)
Connections:
- J101 pad 2: VCC -> +3.3V
- J101 pad 25: unconnected-(J101-Pin_25-Pad25) -> calliope_M0+
- J101 pad 27: unconnected-(J101-Pin_27-Pad27) -> calliope_M0-
- J101 pad 3: unconnected-(J101-Pin_3-Pad3) -> calliope_P0
Routing:
- net (no net): track 10243.5 -> 0.00 mm, vias 0 -> 1
- net +3.3V: track 0.00 -> 62.4 mm, vias 0 -> 3
- net GND: track 0.00 -> 55.3 mm, vias 0 -> 20
- net Net-(R101-Pad1): track 0.00 -> 50.6 mm, vias 0 -> 5
- net calliope_P0: track 0.00 -> 37.5 mm, vias 0 -> 2
- net Net-(D103-A): track 0.00 -> 36.1 mm, vias 0 -> 3
- net Net-(D107-K): track 0.00 -> 17.9 mm, vias 0 -> 1
- net +5V_USB: track 0.00 -> 17.6 mm, vias 0 -> 1
- net calliope_M0-: track 0.00 -> 15.6 mm, vias 0 -> 1
- net calliope_M0+: track 0.00 -> 15.6 mm, vias 0 -> 1
- net Net-(D103-K): track 0.00 -> 14.2 mm, vias 0 -> 1
- net Net-(U104-Out): track 0.00 -> 12.3 mm, vias 0 -> 2
- net Net-(SW102-B-Pad2): track 0.00 -> 11.5 mm, vias 0 -> 2
- net Net-(D102-K): track 0.00 -> 11.4 mm, vias 0 -> 2
- net Net-(U102A-+): track 0.00 -> 6.41 mm, vias 0 -> 1
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- added copper zone on B.Cu, net GND
- added copper zone on F.Cu, net GND
Other:
- board outline added: 49 x 67 mm

Commit message: Finished calliope board! Ready to export production files.
Parts:
- added G***: LOGO, logos:uc2-hexa-cubes_coarse_5mm, B.Cu at (97.8, 87.2)
- moved R10 2.44 mm to (92.6, 86.7), turned to 180 degrees
- moved D11 2.11 mm to (90.7, 86.1)
- moved D8 1.44 mm to (90.7, 87.3)
- renumbered C401 to C1, C102 to C2, C103 to C3, C405 to C4, C101 to C5, D1904 to D1, D103 to D10, D109 to D11, D106 to D2, D101 to D3, D102 to D4, D107 to D5, D108 to D6, D105 to D7, D1905 to D8, D104 to D9, J102 to J1, J101 to J2, R103 to R1, R109 to R10, R108 to R2, R102 to R3, R105 to R4, R106 to R5, R107 to R6, R110 to R7, R111 to R8, R101 to R9, SW102 to SW1, TH101 to TH1, TP106 to TP1, TP401 to TP10, TP108 to TP11, TP107 to TP12, TP402 to TP13, TP403 to TP14, TP109 to TP15, TP110 to TP16, TP111 to TP17, TP118 to TP18, TP119 to TP19, TP101 to TP2, TP112 to TP20, TP113 to TP21, TP117 to TP22, TP123 to TP23, TP124 to TP24, TP126 to TP25, TP122 to TP26, TP125 to TP27, TP127 to TP28, TP121 to TP29, TP102 to TP3, TP128 to TP30, TP129 to TP31, TP120 to TP32, TP103 to TP4, TP104 to TP5, TP105 to TP6, TP115 to TP7, TP116 to TP8, TP114 to TP9, U102 to U1, U104 to U2, U401 to U3, U105 to U4
Connections:
- J2 pad 30: unconnected-(J101-Pin_30-Pad30) -> GND
Routing:
- net Net-(D10-K): track 14.2 -> 10.2 mm
- net GND: track 55.3 -> 58.0 mm, vias 20 -> 22
- net Net-(R10-Pad1): track 50.6 -> 49.7 mm, vias 5 -> 6
- net (no net): vias 1 -> 0
Other:
- board text added: "Glue everything to insert with this side"
- board text added: "Glue mirror here"
- board text added: "HEATING"
- board text added: "Heater traces: Length: 5916 mm Width: 0.2 mm Copper layer: 1 oz/cuft Resistance: 14-17 Ohm (PTC)"
- board text added: "M0"
- board text added: "M0+"
- board text added: "M0-"
- board text added: "NTC on Pin P0"
- board text added: "Power:"
- board text added: "USB"
- board text added: "calliope-mirror-heater christiankuttke 2025-09-22; Rev. A openUC2 GmbH"
- board text added: "~4.6V across heater. 80°C overtemperature cutoff, 2°K hysteresis."
